File: kicad/prototypes/1/avr.sch (KiCad schematic (older format))
At the start: 15 parts, among them IC1 ATTINY841-SSU, P1 USB_B, P2 CONN_01X06, P3 CONN_01X02, P4 CONN_01X02, Y1 Crystal

Commit message: Updated to new kicad
Parts:
- P1: symbol USB_B -> USB_B-RESCUE-prototype1
Changed lines of the file:
@@
 EESchema Schematic File Version 2
+LIBS:prototype1-rescue
 LIBS:power
 LIBS:device
@@
 AVR_TXD
 $Comp
-L USB_B P1
+L USB_B-RESCUE-prototype1 P1
 U 1 1 5839FABB
 P 8250 2950
+AR Path="/5839FABB" Ref="P1"  Part="1"
+AR Path="/5839DEEE/5839FABB" Ref="P1"  Part="1"
 F 0 "P1" H 8450 2750 50  0000 C CNN
 F 1 "USB_B" H 8200 3150 50  0000 C CNN
